Commit message: 9.29 update daily notes -- gazebo

File: ros2/chapt6_ws/install/fishbot_description/share/fishbot_description/urdf/fishbot/actuator/caster.urdf.xacro (robot description, xacro)
@@ -1,4 +1,5 @@
 <?xml version="1.0"?>
 <robot xmlns:xacro="http://www.ros.org/wiki/xacro">
+    <xacro:include filename="$(find fishbot_description)/urdf/fishbot/common_inertia.xacro"/>
     <xacro:macro name="caster_xacro" params="caster_name xyz">
         <link name="${caster_name}_link">
@@ -17,4 +18,18 @@
                 </material>
             </visual>
+            <collision>
+                <!-- 沿着自身几何中心的偏移和旋转量 -->
+                <origin xyz="0.0 0.0 0.0" rpy="0.0 0.0 0.0"/>
+                <!-- 几何形状 -->
+                <geometry>
+                    <sphere radius="0.016"/>
+                </geometry>
+                <!-- 材质和颜色描述 -->
+                <material name="yellow">
+                    <!-- 红绿蓝透明度 -->
+                    <color rgba="1.0 1.0 0.0 0.8"/>
+                </material>
+            </collision>
+            <xacro:sphere_inertia m="0.05" r="0.016" />
         </link>
         <!-- 机器人的关节 用于组合机器人的部件 -->

File: ros2/chapt6_ws/install/fishbot_description/share/fishbot_description/urdf/fishbot/actuator/wheel.urdf.xacro (robot description, xacro)
@@ -1,4 +1,5 @@
 <?xml version="1.0"?>
 <robot xmlns:xacro="http://www.ros.org/wiki/xacro">
+    <xacro:include filename="$(find fishbot_description)/urdf/fishbot/common_inertia.xacro"/>
     <xacro:macro name="wheel_xacro" params="wheel_name xyz">
         <link name="${wheel_name}_link">
@@ -17,4 +18,18 @@
                 </material>
             </visual>
+            <collision>
+                <!-- 沿着自身几何中心的偏移和旋转量 -->
+                <origin xyz="0.0 0.0 0.0" rpy="1.57079 0.0 0.0"/>
+                <!-- 几何形状 -->
+                <geometry>
+                    <cylinder radius="0.032" length="0.04"/>
+                </geometry>
+                <!-- 材质和颜色描述 -->
+                <material name="yellow">
+                    <!-- 红绿蓝透明度 -->
+                    <color rgba="1.0 1.0 0.0 0.8"/>
+                </material>
+            </collision>
+            <xacro:cylinder_inertia m="0.05" r="0.032" h="0.04" />
         </link>
         <!-- 机器人的关节 用于组合机器人的部件 -->

File: ros2/chapt6_ws/install/fishbot_description/share/fishbot_description/urdf/fishbot/base.urdf.xacro (robot description, xacro)
@@ -1,5 +1,8 @@
 <?xml version="1.0"?>
 <robot xmlns:xacro="http://www.ros.org/wiki/xacro">
+    <xacro:include filename="$(find fishbot_description)/urdf/fishbot/common_inertia.xacro"/>
     <xacro:macro name="base_xacro" params="length radius">
+        <!-- 虚拟部件不需要内容 -->
+        <link name="base_footprint" />
         <link name="base_link">
         <!-- 部件的外观描述 -->
@@ -18,5 +21,25 @@
             </material>
         </visual>
+        <collision>
+            <!-- 沿着自身几何中心的偏移和旋转量 -->
+            <origin xyz="0.0 0.0 0.0" rpy="0.0 0.0 0.0"/>
+            <!-- 几何形状 -->
+            <geometry>
+                <!-- 圆柱体 单位：m -->
+                <cylinder radius="${radius}" length="${length}"/>
+            </geometry>
+            <!-- 材质和颜色描述 -->
+            <material name="white">
+                <!-- 红绿蓝透明度 -->
+                <color rgba="1.0 1.0 1.0 0.5"/>
+            </material>
+        </collision>
+        <xacro:cylinder_inertia m="1.0" r="${radius}" h="${length}" />
     </link>
+    <joint name="joint_name" type="fixed">
+        <origin xyz="0.0 0.0 ${length/2.0+0.032-0.001}" rpy="0.0 0.0 0.0"/>
+        <parent link="base_footprint"/>
+        <child link="base_link"/>
+    </joint>
     </xacro:macro>
 </robot>

File: ros2/chapt6_ws/install/fishbot_description/share/fishbot_description/urdf/fishbot/sensor/camera.urdf.xacro (robot description, xacro)
@@ -1,4 +1,5 @@
 <?xml version="1.0"?>
 <robot xmlns:xacro="http://www.ros.org/wiki/xacro">
+    <xacro:include filename="$(find fishbot_description)/urdf/fishbot/common_inertia.xacro"/>
     <xacro:macro name="camera_xacro" params="xyz">
         <link name="camera_link">
@@ -18,4 +19,19 @@
                 </material>
             </visual>
+            <collision>
+                <!-- 沿着自身几何中心的偏移和旋转量 -->
+                <origin xyz="0.0 0.0 0.0" rpy="0.0 0.0 0.0"/>
+                <!-- 几何形状 -->
+                <geometry>
+                    <!-- 长宽高 m -->
+                    <box size="0.02 0.10 0.02"/>
+                </geometry>
+                <!-- 材质和颜色描述 -->
+                <material name="black">
+                    <!-- 红绿蓝透明度 -->
+                    <color rgba="0.0 0.0 0.0 0.5"/>
+                </material>
+            </collision>
+            <xacro:box_inertia m="0.1" w="0.02" h="0.10" d="0.02" />
         </link>
         <!-- 机器人的关节 用于组合机器人的部件 -->

File: ros2/chapt6_ws/install/fishbot_description/share/fishbot_description/urdf/fishbot/sensor/imu.urdf.xacro (robot description, xacro)
@@ -1,4 +1,5 @@
 <?xml version="1.0"?>
 <robot xmlns:xacro="http://www.ros.org/wiki/xacro">
+    <xacro:include filename="$(find fishbot_description)/urdf/fishbot/common_inertia.xacro"/>
     <xacro:macro name="imu_xacro" params="xyz">
         <link name="imu_link">
@@ -18,4 +19,19 @@
                 </material>
             </visual>
+            <collision>
+                <!-- 沿着自身几何中心的偏移和旋转量 -->
+                <origin xyz="0.0 0.0 0.0" rpy="0.0 0.0 0.0"/>
+                <!-- 几何形状 -->
+                <geometry>
+                    <!-- 长宽高 m -->
+                    <box size="0.02 0.02 0.02"/>
+                </geometry>
+                <!-- 材质和颜色描述 -->
+                <material name="black">
+                    <!-- 红绿蓝透明度 -->
+                    <color rgba="0.0 0.0 0.0 0.5"/>
+                </material>
+            </collision>
+            <xacro:box_inertia m="0.02" w="0.02" h="0.02" d="0.02" />
         </link>
         <!-- 机器人的关节 用于组合机器人的部件 -->

File: ros2/chapt6_ws/install/fishbot_description/share/fishbot_description/urdf/fishbot/sensor/laser.urdf.xacro (robot description, xacro)
@@ -1,4 +1,5 @@
 <?xml version="1.0"?>
 <robot xmlns:xacro="http://www.ros.org/wiki/xacro">
+    <xacro:include filename="$(find fishbot_description)/urdf/fishbot/common_inertia.xacro"/>
     <xacro:macro name="laser_xacro" params="xyz">
         <!-- 雷达支撑杆 -->
@@ -19,4 +20,19 @@
                 </material>
             </visual>
+            <collision>
+                <!-- 沿着自身几何中心的偏移和旋转量 -->
+                <origin xyz="0.0 0.0 0.0" rpy="0.0 0.0 0.0"/>
+                <!-- 几何形状 -->
+                <geometry>
+                    <!-- 长宽高 m -->
+                    <cylinder radius="0.01" length="0.10"/>
+                </geometry>
+                <!-- 材质和颜色描述 -->
+                <material name="white">
+                    <!-- 红绿蓝透明度 -->
+                    <color rgba="0.0 0.0 0.0 1.0"/>
+                </material>
+            </collision>
+            <xacro:cylinder_inertia m="0.05" r="0.01" h="0.10" />
         </link>
         <link name="laser_link">
@@ -36,4 +52,19 @@
                 </material>
             </visual>
+            <collision>
+                <!-- 沿着自身几何中心的偏移和旋转量 -->
+                <origin xyz="0.0 0.0 0.0" rpy="0.0 0.0 0.0"/>
+                <!-- 几何形状 -->
+                <geometry>
+                    <!-- 长宽高 m -->
+                    <cylinder radius="0.02" length="0.02"/>
+                </geometry>
+                <!-- 材质和颜色描述 -->
+                <material name="white">
+                    <!-- 红绿蓝透明度 -->
+                    <color rgba="0.0 0.0 0.0 1.0"/>
+                </material>
+            </collision>
+            <xacro:cylinder_inertia m="0.10" r="0.02" h="0.02" />
         </link>
         <!-- 机器人的关节 用于组合机器人的部件 -->
